File: PCB/pendulumRobotModule.sch (KiCad schematic (older format))
At the start: 34 parts, among them J1 Conn_01x02_Female, J2 conn_3x4, J3 Conn_01x02_Male, J4 Conn_01x04_Female, J5 conn_3x3, J6 Conn_01x02_Male, J7 Conn_01x04_Female, J8 Conn_01x02_Male, SW1 SW_SPDT, U1 ESP32-devKit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

Commit message: Some slight updates to PCB, also updated readme for PCB
Parts:
- added C7: 10u 50V, Capacitor_SMD:C_1206_3216Metric, symbol Device:C
- added C8: 22u 10V, Capacitor_SMD:C_0805_2012Metric, symbol Device:C
- added U4: R-78E5.0-0.5, Converter_DCDC:Converter_DCDC_RECOM_R-78E-0.5_THT, symbol Regulator_Switching:R-78E5.0-0.5
- C1, C3, C5: footprint Capacitors_SMD:C_0805_HandSoldering -> Capacitor_SMD:C_0805_2012Metric
- D1, D2: footprint LED_THT:LED_D5.0mm -> mylib:LED_D5.0mm_Horizontal
- R1, R10, R2, R3, R4, R5, R6, R7, R8, R9: footprint Resistors_SMD:R_0805_HandSoldering -> Resistor_SMD:R_0805_2012Metric
- SW1: footprint mylib:switch_slider_SPDT_angled -> mylib:switch_slider_SPDT
Connections:
- wire segments 194 -> 202
Changed lines of the file:
@@
 F 0 "R5" H 4670 2196 50  0000 L CNN
 F 1 "100k" H 4670 2105 50  0000 L CNN
-F 2 "Resistors_SMD:R_0805_HandSoldering" V 4530 2150 50  0001 C CNN
+F 2 "Resistor_SMD:R_0805_2012Metric" V 4530 2150 50  0001 C CNN
 F 3 "~" H 4600 2150 50  0001 C CNN
 	1    4600 2150
@@
 F 0 "R6" H 4670 2596 50  0000 L CNN
 F 1 "3k3" H 4670 2505 50  0000 L CNN
-F 2 "Resistors_SMD:R_0805_HandSoldering" V 4530 2550 50  0001 C CNN
+F 2 "Resistor_SMD:R_0805_2012Metric" V 4530 2550 50  0001 C CNN
 F 3 "~" H 4600 2550 50  0001 C CNN
 	1    4600 2550
@@
 F 0 "C3" H 5065 2596 50  0000 L CNN
 F 1 "1u" H 5065 2505 50  0000 L CNN
-F 2 "Capacitors_SMD:C_0805_HandSoldering" H 4988 2400 50  0001 C CNN
+F 2 "Capacitor_SMD:C_0805_2012Metric" H 4988 2400 50  0001 C CNN
 F 3 "~" H 4950 2550 50  0001 C CNN
 	1    4950 2550
@@
 F 0 "R1" H 1470 6396 50  0000 L CNN
 F 1 "3k3" H 1470 6305 50  0000 L CNN
-F 2 "Resistors_SMD:R_0805_HandSoldering" V 1330 6350 50  0001 C CNN
+F 2 "Resistor_SMD:R_0805_2012Metric" V 1330 6350 50  0001 C CNN
 F 3 "~" H 1400 6350 50  0001 C CNN
 	1    1400 6350
@@
 F 0 "R2" H 1470 6796 50  0000 L CNN
 F 1 "3k3" H 1470 6705 50  0000 L CNN
-F 2 "Resistors_SMD:R_0805_HandSoldering" V 1330 6750 50  0001 C CNN
+F 2 "Resistor_SMD:R_0805_2012Metric" V 1330 6750 50  0001 C CNN
 F 3 "~" H 1400 6750 50  0001 C CNN
 	1    1400 6750
@@
 F 0 "C1" H 1915 6796 50  0000 L CNN
 F 1 "1u" H 1915 6705 50  0000 L CNN
-F 2 "Capacitors_SMD:C_0805_HandSoldering" H 1838 6600 50  0001 C CNN
+F 2 "Capacitor_SMD:C_0805_2012Metric" H 1838 6600 50  0001 C CNN
 F 3 "~" H 1800 6750 50  0001 C CNN
 	1    1800 6750
@@
 F 0 "R3" H 3420 6546 50  0000 L CNN
 F 1 "3k3" H 3420 6455 50  0000 L CNN
-F 2 "Resistors_SMD:R_0805_HandSoldering" V 3280 6500 50  0001 C CNN
+F 2 "Resistor_SMD:R_0805_2012Metric" V 3280 6500 50  0001 C CNN
 F 3 "~" H 3350 6500 50  0001 C CNN
 	1    3350 6500
@@
 F 0 "R4" H 3670 6546 50  0000 L CNN
 F 1 "3k3" H 3670 6455 50  0000 L CNN
-F 2 "Resistors_SMD:R_0805_HandSoldering" V 3530 6500 50  0001 C CNN
+F 2 "Resistor_SMD:R_0805_2012Metric" V 3530 6500 50  0001 C CNN
 F 3 "~" H 3600 6500 50  0001 C CNN
 	1    3600 6500
@@
 F 0 "C5" H 4615 4146 50  0000 L CNN
 F 1 "100n" H 4615 4055 50  0000 L CNN
-F 2 "Capacitors_SMD:C_0805_HandSoldering" H 4538 3950 50  0001 C CNN
+F 2 "Capacitor_SMD:C_0805_2012Metric" H 4538 3950 50  0001 C CNN
 F 3 "~" H 4500 4100 50  0001 C CNN
 	1    4500 4100
@@
 F 0 "R7" H 5020 4146 50  0000 L CNN
 F 1 "3k3" H 5020 4055 50  0000 L CNN
-F 2 "Resistors_SMD:R_0805_HandSoldering" V 4880 4100 50  0001 C CNN
+F 2 "Resistor_SMD:R_0805_2012Metric" V 4880 4100 50  0001 C CNN
 F 3 "~" H 4950 4100 50  0001 C CNN
 	1    4950 4100
@@
 F 0 "R8" H 770 4046 50  0000 L CNN
 F 1 "100k" H 770 3955 50  0000 L CNN
-F 2 "Resistors_SMD:R_0805_HandSoldering" V 630 4000 50  0001 C CNN
+F 2 "Resistor_SMD:R_0805_2012Metric" V 630 4000 50  0001 C CNN
 F 3 "~" H 700 4000 50  0001 C CNN
 	1    700  4000
@@
 F 0 "SW1" H 2800 2135 50  0000 C CNN
 F 1 "SW_SPDT" H 2800 2044 50  0000 C CNN
-F 2 "mylib:switch_slider_SPDT_angled" H 2800 1850 50  0001 C CNN
+F 2 "mylib:switch_slider_SPDT" H 2800 1850 50  0001 C CNN
 F 3 "~" H 2800 1850 50  0001 C CNN
 	1    2800 1850
@@
 F 0 "D1" V 889 5233 50  0000 R CNN
 F 1 "LED" V 798 5233 50  0000 R CNN
-F 2 "LED_THT:LED_D5.0mm" H 850 5350 50  0001 C CNN
+F 2 "mylib:LED_D5.0mm_Horizontal" H 850 5350 50  0001 C CNN
 F 3 "~" H 850 5350 50  0001 C CNN
 	1    850  5350
@@
 F 0 "R9" H 920 4946 50  0000 L CNN
 F 1 "100k" H 920 4855 50  0000 L CNN
-F 2 "Resistors_SMD:R_0805_HandSoldering" V 780 4900 50  0001 C CNN
+F 2 "Resistor_SMD:R_0805_2012Metric" V 780 4900 50  0001 C CNN
 F 3 "~" H 850 4900 50  0001 C CNN
 	1    850  4900
@@
 F 0 "D2" V 1189 5233 50  0000 R CNN
 F 1 "LED" V 1098 5233 50  0000 R CNN
-F 2 "LED_THT:LED_D5.0mm" H 1150 5350 50  0001 C CNN
+F 2 "mylib:LED_D5.0mm_Horizontal" H 1150 5350 50  0001 C CNN
 F 3 "~" H 1150 5350 50  0001 C CNN
 	1    1150 5350
@@
 F 0 "R10" H 1220 4946 50  0000 L CNN
 F 1 "100k" H 1220 4855 50  0000 L CNN
-F 2 "Resistors_SMD:R_0805_HandSoldering" V 1080 4900 50  0001 C CNN
+F 2 "Resistor_SMD:R_0805_2012Metric" V 1080 4900 50  0001 C CNN
 F 3 "~" H 1150 4900 50  0001 C CNN
 	1    1150 4900
@@
 Wire Wire Line
 	3000 1950 3200 1950
+Wire Wire Line
+	5250 950  5000 950
+Wire Wire Line
+	5000 950  5000 1050
+$Comp
+L power:GND #PWR0131
+U 1 1 632457A8
+P 5000 1350
+F 0 "#PWR0131" H 5000 1100 50  0001 C CNN
+F 1 "GND" H 5005 1177 50  0000 C CNN
+F 2 "" H 5000 1350 50  0001 C CNN
+F 3 "" H 5000 1350 50  0001 C CNN
+	1    5000 1350
+	1    0    0    -1
+$EndComp
+$Comp
+L power:GND #PWR0132
+U 1 1 63245B55
+P 5550 1350
+F 0 "#PWR0132" H 5550 1100 50  0001 C CNN
+F 1 "GND" H 5555 1177 50  0000 C CNN
+F 2 "" H 5550 1350 50  0001 C CNN
+F 3 "" H 5550 1350 50  0001 C CNN
+	1    5550 1350
+	1    0    0    -1
+$EndComp
+$Comp
+L power:GND #PWR0133
+U 1 1 63245D3C
+P 6000 1350
+F 0 "#PWR0133" H 6000 1100 50  0001 C CNN
+F 1 "GND" H 6005 1177 50  0000 C CNN
+F 2 "" H 6000 1350 50  0001 C CNN
+F 3 "" H 6000 1350 50  0001 C CNN
+	1    6000 1350
+	1    0    0    -1
+$EndComp
+Wire Wire Line
+	5550 1250 5550 1350
+Wire Wire Line
+	5850 950  6000 950
+Wire Wire Line
+	6000 950  6000 1050
+$Comp
+L power:+5V #PWR0134
+U 1 1 6325C9A8
+P 6000 900
+F 0 "#PWR0134" H 6000 750 50  0001 C CNN
+F 1 "+5V" H 6015 1073 50  0000 C CNN
+F 2 "" H 6000 900 50  0001 C CNN
+F 3 "" H 6000 900 50  0001 C CNN
+	1    6000 900
+	1    0    0    -1
+$EndComp
+Wire Wire Line
+	6000 900  6000 950
+Connection ~ 6000 950
+Wire Wire Line
+	5000 950  4850 950
+Wire Wire Line
+	4850 950  4850 900
+Connection ~ 5000 950
+$Comp
+L power:+24V #PWR0135
+U 1 1 6327396F
+P 4850 900
+F 0 "#PWR0135" H 4850 750 50  0001 C CNN
+F 1 "+24V" H 4865 1073 50  0000 C CNN
+F 2 "" H 4850 900 50  0001 C CNN
+F 3 "" H 4850 900 50  0001 C CNN
+	1    4850 900
+	1    0    0    -1
+$EndComp
+$Comp
+L Regulator_Switching:R-78E5.0-0.5 U4
+U 1 1 6322C7A5
+P 5550 950
+F 0 "U4" H 5550 1192 50  0000 C CNN
+F 1 "R-78E5.0-0.5" H 5550 1101 50  0000 C CNN
+F 2 "Converter_DCDC:Converter_DCDC_RECOM_R-78E-0.5_THT" H 5600 700 50  0001 L CIN
+F 3 "https://www.recom-power.com/pdf/Innoline/R-78Exx-0.5.pdf" H 5550 950 50  0001 C CNN
+	1    5550 950
+	1    0    0    -1
+$EndComp
+$Comp
+L Device:C C7
+U 1 1 632762D9
+P 5000 1200
+F 0 "C7" H 5115 1246 50  0000 L CNN
+F 1 "10u 50V" H 5115 1155 50  0000 L CNN
+F 2 "Capacitor_SMD:C_1206_3216Metric" H 5038 1050 50  0001 C CNN
+F 3 "~" H 5000 1200 50  0001 C CNN
+	1    5000 1200
+	1    0    0    -1
+$EndComp
+$Comp
+L Device:C C8
+U 1 1 632766A1
+P 6000 1200
+F 0 "C8" H 6115 1246 50  0000 L CNN
+F 1 "22u 10V" H 6115 1155 50  0000 L CNN
+F 2 "Capacitor_SMD:C_0805_2012Metric" H 6038 1050 50  0001 C CNN
+F 3 "~" H 6000 1200 50  0001 C CNN
+	1    6000 1200
+	1    0    0    -1
+$EndComp
 $EndSCHEMATC
